Commit message: working dummy model of iisy

File: urdf/iisy11_model.urdf (robot description, URDF)
Before this commit: robot LBRiisy11R1300, 11 links, 10 joints
Links:
- link base_link_inertia: geometry collision mesh filename=package://iisy11_model/meshes/LBRiisy11R1300/collision/base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; visual mesh filename=package://iisy11_model/meshes/LBRiisy11R1300/visual/base_li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
- link link_1: geometry collision mesh filename=package://iisy11_model/meshes/LBRiisy11R1300/collision/link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; visual mesh filename=package://iisy11_model/meshes/LBRiisy11R1300/visual/link_1.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
- link link_2: geometry collision mesh filename=package://iisy11_model/meshes/LBRiisy11R1300/collision/link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; visual mesh filename=package://iisy11_model/meshes/LBRiisy11R1300/visual/link_2.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
- link link_3: geometry collision mesh filename=package://iisy11_model/meshes/LBRiisy11R1300/collision/link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; visual mesh filename=package://kuka_lbr_iisy_support/meshes/LBRiisy11R1300/visua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
